File: kicad/lpwa-node.kicad_sch (KiCad schematic)
At the start: 31 parts, among them J1 USB_C_ESP, SW1 BOOT, SW2 RESET, SW3 BOOT, U1 ESP32-C3-WROOM-02, U3 BH-AA-B6AA044, U4 USBLC6-2SC6, U5 AHT20, U8 TPS7A0230PDBVR

Commit message: Draft
Parts:
- removed R12, R16: 10k, Resistor_SMD:R_0603_1608Metric, symbol Device:R_Small
- removed R4: 2.7k, Resistor_SMD:R_0603_1608Metric, symbol Device:R_Small
- removed SW2: RESET, lighthouse_footprints:SW_SPST_PTS810, symbol Switch:SW_Push
- removed TP1: GND, TestPoint:TestPoint_Pad_D1.0mm, symbol Connector:TestPoint_Small
- removed TP2: RESET, lighthouse_footprints:TestPoint_Pad_D1.0mm_no_court, symbol Connector:TestPoint_Small
- added J2: I2C, Connector_PinHeader_2.54mm:PinHeader_2x02_P2.54mm_Vertical_SMD, symbol Connector:Conn_01x04_Pin
- added J3: USB to VBAT, Connector_PinHeader_2.54mm:PinHeader_1x03_P2.54mm_Vertical, symbol Connector:Conn_01x03_Pin
- added JP1: RESET, Jumper:SolderJumper-2_P1.3mm_Open_RoundedPad1.0x1.5mm, symbol Jumper:Jumper_2_Small_Open
- added R6, R7: 5.1k, Resistor_SMD:R_0603_1608Metric, symbol Device:R_Small
- added TP5: IO20/RXD, TestPoint:TestPoint_Pad_D1.5mm, symbol Connector:TestPoint_Small
- added TP6: IO21/TXD, TestPoint:TestPoint_Pad_D1.5mm, symbol Connector:TestPoint_Small
- D1: value LED White KT-0603W -> LED Amber BL-HJC36G-AV-TRB; LCSC Part # C2290 -> C165983
- R8: renamed from R18; LCSC Part # (none) -> C22935
- R9: renamed from R17; LCSC Part # (none) -> C22935
- SW1: footprint Button_Switch_SMD:SW_Push_1P1T_XKB_TS-1187A -> lpwa-node:SW_Push_1P1T_XKB_TS-1187A
- SW2: renamed from SW3; value BOOT -> USER; footprint Button_Switch_SMD:SW_Push_1P1T_XKB_TS-1187A -> lpwa-node:SW_Push_1P1T_XKB_TS-1187A
- renumbered C25 to C1, C26 to C2, C24 to C3, C18 to C4, C28 to C5, C19 to C6, C13 to C7, D5 to D2, D6 to D3, R5 to R4, R6 to R5, U8 to U1, U4 to U2, U1 to U3, U5 to U4, U3 to U5
Connections:
- net +5V is gone; now on net +BATT: C1.2, U1.1 (IN), U1.3 (EN)
- net +3V3: now also J2.1 (Pin_1), R6.2, R7.2
- net +BATT: now also J3.3 (Pin_3)
- net EN: now also JP1.2 (B)
- net GND: now also J2.2 (Pin_2), J3.2 (Pin_2), JP1.1 (A)
- net SCL: now also J2.3 (Pin_3)
- net SDA: now also J2.4 (Pin_4)
- net USB_ESP_+5V: now also J3.1 (Pin_1)
- net at D1.2 (A): now also R6.1, R7.1
- net RX/20: no longer names the net of U3.11 (IO20/RXD)
- net RX/20: now also TP5.1
- net STATUS renamed ESP_SIM_STATUS
- net TX/21: no longer names the net of U3.12 (IO21/TXD)
- net TX/21: now also TP6.1
Other:
- added sheet RF (rf.kicad_sch)
- added sheet SIM7080 (sim7080.kicad_sch)
- note removed: "Excluded"
- moved on the sheet: D1

Commit message: Draft
Parts:
- removed J2: I2C, Connector_PinHeader_2.54mm:PinHeader_2x02_P2.54mm_Vertical_SMD, symbol Connector:Conn_01x04_Pin
- removed J3: USB to VBAT, Connector_PinHeader_2.54mm:PinHeader_1x03_P2.54mm_Vertical, symbol Connector:Conn_01x03_Pin
- added C20, C21: 10µF, Capacitor_SMD:C_0603_1608Metric, symbol Device:C_Small
- added JP11: VSYS_BYPASS, Jumper:SolderJumper-2_P1.3mm_Open_RoundedPad1.0x1.5mm, symbol Jumper:Jumper_2_Small_Open
- added R18: 100k, Resistor_SMD:R_0603_1608Metric, symbol Device:R_Small
- added R19: 732k, Resistor_SMD:R_0603_1608Metric, symbol Device:R_Small
- added R20: 1M, Resistor_SMD:R_0603_1608Metric, symbol Device:R_Small
- added R21: 10k, Resistor_SMD:R_0603_1608Metric, symbol Device:R_Small
- added TP10: SDA, TestPoint:TestPoint_Pad_D1.5mm, symbol Connector:TestPoint_Small
- added TP11: USB_5V, TestPoint:TestPoint_Pad_D1.5mm, symbol Connector:TestPoint_Small
- added TP12: VSYS, TestPoint:TestPoint_Pad_D1.5mm, symbol Connector:TestPoint_Small
- added TP7: 3V0, TestPoint:TestPoint_Pad_D1.5mm, symbol Connector:TestPoint_Small
- added TP8: GND, TestPoint:TestPoint_Pad_D1.5mm, symbol Connector:TestPoint_Small
- added TP9: SCL, TestPoint:TestPoint_Pad_D1.5mm, symbol Connector:TestPoint_Small
- added U10, U11: LM66100DCK, Package_TO_SOT_SMD:SOT-363_SC-70-6, symbol Power_Management:LM66100DCK
- added U9: TLV75901PDRVR, lpwa-node:WSON-6_L2.0-W2.0-P0.65-TL-EP, symbol lpwa-node:TLV75901PDRVR
Connections:
- net GND: now also C20.1, C21.1, R18.2, R20.2, TP8.1, U10.2 (GND), U10.5 (ST), U11.2 (GND), U9.3 (GND), U9.7 (EP)
- net SCL: now also TP9.1
- net SDA: now also TP10.1
- net USB_ESP_+5V: now also C21.2, R21.1, TP11.1, U9.4 (EN), U9.6 (IN)
- net +3V3 renamed 3V0
- net 3V0: now also TP7.1
- net +BATT renamed BATTERY
- net BATTERY: now also JP11.1 (A), U10.1 (VIN); no longer C1.2, U1.1 (IN), U1.3 (EN)
- new net: R20.1, R21.2, U10.3 (~{CE}), U11.5 (ST)
- new net: R18.1, R19.2, U9.2 (FB)
- new net USB_4V6: C20.2, R19.1, U11.1 (VIN), U9.1 (OUT)
- new net VSYS: C1.2, JP11.2 (B), TP12.1, U1.1 (IN), U1.3 (EN), U10.6 (VOUT), U11.3 (~{CE}), U11.6 (VOUT)
Other:
- moved on the sheet: C7, D3, R8, R9, U5

Commit message: Draft
Parts:
- added R23: 1M, Resistor_SMD:R_0603_1608Metric, symbol Device:R_Small
- added R24: 732k, Resistor_SMD:R_0603_1608Metric, symbol Device:R_Small
Connections:
- net GND: now also R23.2
- net USB_ESP_+5V: now also R24.1
- net ESP_SIM_RI renamed ESP_USB_SENSE
- net ESP_USB_SENSE: now also R23.1, R24.2
Other:
- moved on the sheet: C1, C3, C7, R8, R9, TP10, TP11, TP12, TP7, TP8, TP9, U1

Commit message: First orderable version
Parts:
- added D7, D8, D9: ESD5Z3.3T1G, Diode_SMD:D_SOD-523, symbol Diode:ESD5Zxx
- added R25: 100k, Resistor_SMD:R_0603_1608Metric, symbol Device:R_Small
- C6: value 100nF -> 10µF; LCSC Part # C14663 -> C19702
Connections:
- net 3V0: now also D7.1 (K), R25.1
- net ESP_BTN: now also R25.2
- net GND: now also D7.2 (A), D8.2 (A), D9.2 (A)
- net SCL: now also D9.1 (K)
- net SDA: now also D8.1 (K)
Other:
- moved on the sheet: C6, U4

Commit message: Optimize for manufacturing, add part numbers
Parts:
- added J2: Manufacturing Jig, lpwa-node:TestHeader_1x05_P2.54mm, symbol Connector:Conn_01x05_Socket
- C4, C7: LCSC Part # C14663 -> C161115
- D2, D7, D8, D9: LCSC Part # (none) -> C61148
- D3: LCSC Part # (none) -> C82044
- JP1, TP10, TP11, TP12, TP5, TP6, TP7, TP8, TP9: now left out of the parts list
- JP11: value VSYS_BYPASS -> BYPASS; now left out of the parts list
- U10, U11: LCSC Part # (none) -> C2869734
- U5: LCSC Part C19184082 -> (none); LCSC Part # (none) -> C19184082; MANUFACTURER (none) -> MYOUNG(美阳); Manufacturer MYOUNG(美阳) -> (none)
- U9: LCSC Part C544759 -> (none); LCSC Part # (none) -> C544759; MANUFACTURER (none) -> TI(德州仪器); Manufacturer TI(德州仪器) -> (none)
Connections:
- net 3V0: now also J2.2 (Pin_2)
- net BATTERY: now also J2.4 (Pin_4)
- net GND: now also J2.1 (Pin_1), J2.5 (Pin_5)
- net VSYS: now also J2.3 (Pin_3)

Commit message: Release A
Parts:
- added T1, T2, T3, T4: Tab, PCM_kikit:Tab, symbol PCM_kikit:Tab
- SW1: LCSC Part # C318885 -> C480267
- SW2: LCSC Part # C318884 -> C480267
