File: kicad/rf.kicad_sch (KiCad schematic)
At the start: 14 parts, among them J4 MEAS, J5 LTE, J7 GNSS

Commit message: Draft
Parts:
- removed C14: DNP, Capacitor_SMD:C_0402_1005Metric, symbol Device:C_Small
- removed C15: 33pF, Capacitor_SMD:C_0402_1005Metric, symbol Device:C_Small
- removed D4: LXES15AAA1-153, Diode_SMD:D_SOD-923, symbol Diode:ESD9B3.3ST5G
- removed J4: MEAS, Connector_Coaxial:U.FL_Hirose_U.FL-R-SMT-1_Vertical, symbol Connector:Conn_Coaxial_Small
- removed J5: LTE, Connector_Coaxial:U.FL_Hirose_U.FL-R-SMT-1_Vertical, symbol Connector:Conn_Coaxial_Small
- removed R13: R0, Resistor_SMD:R_0402_1005Metric, symbol Device:R_Small
- removed R14: 10R, Resistor_SMD:R_0402_1005Metric, symbol Device:R_Small
- added C18: 33pF, Capacitor_SMD:C_0402_1005Metric, symbol Device:C_Small
- added C19: DNP, Capacitor_SMD:C_0402_1005Metric, symbol Device:C_Small
- added D6: LXES15AAA1-153, Diode_SMD:D_SOD-923, symbol Diode:ESD9B3.3ST5G
- added J6: MEAS, Connector_Coaxial:U.FL_Hirose_U.FL-R-SMT-1_Vertical, symbol Connector:Conn_Coaxial_Small
- added J8: LTE, Connector_Coaxial:U.FL_Hirose_U.FL-R-SMT-1_Vertical, symbol Connector:Conn_Coaxial_Small
- added R16: R0, Resistor_SMD:R_0402_1005Metric, symbol Device:R_Small
- added R17: 10R, Resistor_SMD:R_0402_1005Metric, symbol Device:R_Small
- C16: value DNP -> F; now left out of the parts list
- C17: value F -> DNP
- J7, L1, L2, L3: now left out of the parts list
Connections:
- net GND: now also C17.2, C19.2, D6.1 (A1), J6.2 (Ext), J8.2 (Ext); no longer C16.2
- net SIM_GNSS_ANT: now also C16.1; no longer C17.1
- net SIM_LTE_ANT: now also C17.1, J6.1 (In); no longer C16.1
- net VDD_SIM_EXT: now also R17.2
- net LTE_FILTER_1: now reaches R15.2
- net LTE_FILTER_1: now also C19.1, R16.1
- net GNSS_FILTER_3: now reaches L3.1
- net GNSS_FILTER_3: now also R17.1
- net GNSS_FILTER_2: now reaches J7.1 (In), L3.2
- net GNSS_FILTER_2: now also C18.2
- net GNSS_FILTER_1: now reaches L2.1
- net GNSS_FILTER_1: now also C16.2, C18.1; no longer C17.2
- new net LTE_FILTER_2: D6.2 (A2), J8.1 (In), R16.2
Other:
- note added: "Excluded"

Commit message: Optimize for manufacturing, add part numbers
Parts:
- C17, C19: now left out of the parts list
- D6: footprint Diode_SMD:D_SOD-923 -> Diode_SMD:D_SOD-882
- J6: footprint Connector_Coaxial:U.FL_Hirose_U.FL-R-SMT-1_Vertical -> lpwa-node:U.FL_Hirose_MEAS

Commit message: Release A
Parts:
- J6: now left out of the parts list
